File: hardware/drill_charger.brd (EAGLE design)
At the start: 51.3 x 25.1 mm, 24 parts, among them IC1 7805TV, J1 POWER_JACK, Q1 TIP41C, U1 PIC12LF1572/MF

Commit message: cleanup
Parts:
- added TEMP: (no value), SparkFun-Connectors:1X01
- moved CLK 0.51 mm to (25.9, 12.7)
- moved DATA 0.51 mm to (28.4, 12.7)
- moved GND 0.51 mm to (31.0, 12.7)
- moved 5V 0.51 mm to (33.5, 12.7)
- moved RST 0.51 mm to (36.1, 12.7)
Connections:
- removed net LED: U1.2
- net !LED: now also U1.2
- net TSENSE: now also TEMP.1
Routing:
- net GND: track 142.2 -> 147.2 mm
- net LED: track 3.74 -> 0.00 mm
- net !LED: track 0.00 -> 3.74 mm
- net TSENSE: track 0.00 -> 3.23 mm
- net TX: track 11.9 -> 12.9 mm
- net VSENSE: track 33.7 -> 34.5 mm
- net 5V: track 92.4 -> 91.8 mm

Commit message: Add files via upload
Parts:
- added R6: 10K, resistor:R0805
- IC1: value 7805TV -> SMPS 5v
- moved T1 21.6 mm to (31.8, 20.3), turned to 90 degrees
- moved R1 20.1 mm to (27.9, 18.8), turned to 180 degrees
- moved IC1 5.08 mm to (19.1, 1.27), turned to 180 degrees
- moved D3 4.58 mm to (17.8, 7.62), turned to 180 degrees
- moved R2 2.54 mm to (25.4, 3.56)
- moved R4 1.27 mm to (40.6, 8.89), turned to 0 degrees
- moved B+ 0.25 mm to (41.9, 3.56)
- turned R3 to 180 degrees
Connections:
- net N$1 renamed VBATT
- removed net N$5: Q1.B, R2.2, T1.C
- new net SW: Q1.B, R2.2, R5.1, T1.C
- net !VCTL: no longer R5.1
- net +18V: no longer C2.1
- net 5V: now also R6.1
- net MCLR: now also R6.2
- net N$6: now also C2.1
Routing:
- net SW: track 0.00 -> 53.3 mm
- net N$5: track 29.4 -> 0.00 mm
- net !VCTL: track 36.1 -> 9.53 mm, vias 2 -> 0
- net GND: track 147.2 -> 125.1 mm
- net +18V: track 34.7 -> 19.1 mm
- net 5V: track 91.8 -> 81.3 mm, vias 2 -> 0
- net VSENSE: track 34.5 -> 44.7 mm
- net N$6: track 6.07 -> 13.0 mm
- net N$8: track 1.79 -> 2.40 mm
- added copper zone on layer 16, net VBATT
